File: recruitment.kicad_pcb (KiCad board)
At the start: 2 copper layers, 1 part

Commit message: feat: First commit
Parts:
- added C2: 220uF, Capacitor_SMD:C_0402_1005Metric, F.Cu at (192.5, 105.0)
- added C3: ~, Capacitor_SMD:C_0402_1005Metric, F.Cu at (192.5, 107.5)
- added C4: 0.1uF, Capacitor_SMD:C_0402_1005Metric, F.Cu at (192.5, 110.0)
- added D1: 1N5822, Diode_THT:D_DO-201AD_P15.24mm_Horizontal, F.Cu at (178.0, 101.6)
- added D2: LED, LED_SMD:LED_0201_0603Metric_Pad0.64x0.40mm_HandSolder, F.Cu at (191.0, 117.5)
- added D3: LED, LED_SMD:LED_0201_0603Metric_Pad0.64x0.40mm_HandSolder, F.Cu at (190.9, 120.0)
- added D4: 1N914, Diode_THT:D_DO-35_SOD27_P7.62mm_Horizontal, F.Cu at (184.0, 102.3)
- added J1-ALLEGRO1: Conn_01x02_Pin, Connector_Phoenix_GMSTB:PhoenixContact_GMSTBA_2,5_2-G_1x02_P7.50mm_Horizontal, F.Cu at (187.2, 63.8)
- added J2: Screw_Terminal_01x02, Connector_Phoenix_GMSTB:PhoenixContact_GMSTBA_2,5_2-G_1x02_P7.50mm_Horizontal, F.Cu at (222.2, 63.8)
- added J3: Screw_Terminal_01x02, Connector_Phoenix_GMSTB:PhoenixContact_GMSTBA_2,5_2-G_1x02_P7.50mm_Horizontal, F.Cu at (215.2, 80.8)
- added J4: Screw_Terminal_01x02, Connector_Phoenix_GMSTB:PhoenixContact_GMSTBA_2,5_2-G_1x02_P7.50mm_Horizontal, F.Cu at (204.8, 63.8)
- added J5: Da auto, Connector_Phoenix_GMSTB:PhoenixContact_GMSTBA_2,5_2-G_1x02_P7.50mm_Horizontal, F.Cu at (141.2, 119.7)
- added K1: RAYEX-L90, Relay_THT:Relay_SPDT_RAYEX-L90, F.Cu at (211.4, 125.0)
- added L1: L, Inductor_SMD:L_0805_2012Metric, F.Cu at (183.9, 111.5)
- added Q1: BC337, Package_TO_SOT_THT:TO-92_Inline, F.Cu at (206.7, 91.0)
- added Q2: 2N2219, Package_TO_SOT_THT:TO-92L_Inline, F.Cu at (214.2, 91.1)
- added Q3: 2N3905, Package_TO_SOT_THT:TO-92_Inline, F.Cu at (221.5, 91.0)
- added R1: 470k, Resistor_SMD:R_0201_0603Metric, F.Cu at (194.8, 84.0)
- added R10: 10K, Resistor_SMD:R_0201_0603Metric, F.Cu at (160.7, 128.0)
- added R11: 10k, Resistor_SMD:R_0201_0603Metric, F.Cu at (164.5, 124.0)
- added R12: 10K, Resistor_SMD:R_0201_0603Metric, F.Cu at (164.5, 126.0)
- added R13: 10k, Resistor_SMD:R_0201_0603Metric, F.Cu at (164.7, 128.0)
- added R2: 5k, Resistor_SMD:R_0201_0603Metric, F.Cu at (194.8, 86.0)
- added R3: 10k, Resistor_SMD:R_0201_0603Metric, F.Cu at (195.0, 88.0)
- added R4: 4.2K, Resistor_SMD:R_0201_0603Metric, F.Cu at (195.0, 90.0)
- added R5: 10K, Resistor_SMD:R_0201_0603Metric, F.Cu at (200.0, 84.0)
- added R6: 220, Resistor_SMD:R_0201_0603Metric, F.Cu at (200.0, 86.0)
- added R7: 220, Resistor_SMD:R_0201_0603Metric, F.Cu at (200.0, 88.0)
- added R8: 8K, Resistor_SMD:R_0201_0603Metric, F.Cu at (160.5, 124.0)
- added R9: 2K, Resistor_SMD:R_0201_0603Metric, F.Cu at (160.5, 126.0)
- added SW1: SW_Push, Button_Switch_SMD:SW_SPST_TS-1088-xR020, F.Cu at (193.5, 128.5)
- added U1: LM2596S-5V, Package_TO_SOT_SMD:TO-263-5_TabPin3, F.Cu at (180.5, 120.1)
- added U2: LM358, Package_SO:SOIC-8-1EP_3.9x4.9mm_P1.27mm_EP2.29x3mm, F.Cu at (141.2, 110.9)
- added U2-TPS71533__SC70: U2 - 3,3V, Package_TO_SOT_SMD:SOT-353_SC-70-5, F.Cu at (177.0, 109.0)
- added U3: ACS781xLRTR-050B, Sensor_Current:Allegro_PSOF-7_4.8x6.4mm_P1.60mm, F.Cu at (179.7, 75.0)
- added U4: LM339, Package_TO_SOT_SMD:SOT-23-6, F.Cu at (192.5, 96.0)
- added U5: 4013, Package_DIP:DIP-14_W7.62mm, F.Cu at (203.6, 70.7)
- added U7: TEN20-4823WIN, Converter_DCDC:Converter_DCDC_TRACO_TEN20-xxxx_THT, F.Cu at (148.1, 68.8)
- added U8: AD633JRZ-R7, Package_SO:SOIC-8-1EP_3.9x4.9mm_P1.27mm_EP2.29x3mm, F.Cu at (149.2, 110.9)
- C1: value 1F -> 680uF; footprint Capacitor_SMD:C_0805_2012Metric -> Capacitor_SMD:C_0402_1005Metric
- moved C1 44.0 mm to (192.5, 102.5), turned to 180 degrees
Connections:
- C1 pad 1: Net-(C1-Pad1) -> Net-(J2-Pin_2)
- C1 pad 2: Net-(C1-Pad1) -> GND
Routing:
- net GND: track 0.00 -> 346.8 mm, vias 0 -> 2
- net Net-(J2-Pin_2): track 0.00 -> 95.9 mm, vias 0 -> 2
- net Net-(D4-K): track 0.00 -> 91.6 mm, vias 0 -> 4
- net 5V: track 0.00 -> 84.8 mm, vias 0 -> 6
- net 24/48 V: track 0.00 -> 73.2 mm, vias 0 -> 2
- net Net-(U4A--): track 0.00 -> 70.3 mm, vias 0 -> 2
- net Net-(U5A-R): track 0.00 -> 68.0 mm, vias 0 -> 4
- net Net-(D3-K): track 0.00 -> 66.5 mm
- net Net-(U8-Y1): track 0.00 -> 61.1 mm, vias 0 -> 4
- net Net-(J3-Pin_2): track 0.00 -> 60.7 mm
- net Net-(D4-A): track 0.00 -> 59.8 mm, vias 0 -> 2
- net Net-(C1-Pad1): track 57.5 -> 0.00 mm
- net Net-(U2A--): track 0.00 -> 55.4 mm
- net Net-(Q1-B): track 0.00 -> 53.2 mm, vias 0 -> 4
- net Net-(U2-TPS71533__SC70-OUT): track 0.00 -> 47.6 mm, vias 0 -> 2
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- added copper zone on F.Cu, net GND
