File: recruitment.kicad_sch (KiCad schematic)
At the start: 1 part

Commit message: feat: First commit
Parts:
- added C2: 220uF, Capacitor_SMD:C_0402_1005Metric, symbol Device:C
- added C3: (no value), Capacitor_SMD:C_0402_1005Metric, symbol Device:C
- added C4: 0.1uF, Capacitor_SMD:C_0402_1005Metric, symbol Device:C
- added D1: 1N5822, Diode_THT:D_DO-201AD_P15.24mm_Horizontal, symbol Diode:1N5822
- added D2, D3: LED, LED_SMD:LED_0201_0603Metric_Pad0.64x0.40mm_HandSolder, symbol Device:LED
- added D4: 1N914, Diode_THT:D_DO-35_SOD27_P7.62mm_Horizontal, symbol Diode:1N914
- added J1-ALLEGRO1: Conn_01x02_Pin, Connector_Phoenix_GMSTB:PhoenixContact_GMSTBA_2,5_2-G_1x02_P7.50mm_Horizontal, symbol Connector:Conn_01x02_Pin
- added J2, J3, J4: Screw_Terminal_01x02, Connector_Phoenix_GMSTB:PhoenixContact_GMSTBA_2,5_2-G_1x02_P7.50mm_Horizontal, symbol Connector:Screw_Terminal_01x02
- added J5: Da auto, Connector_Phoenix_GMSTB:PhoenixContact_GMSTBA_2,5_2-G_1x02_P7.50mm_Horizontal, symbol Connector:Screw_Terminal_01x02
- added K1: RAYEX-L90, Relay_THT:Relay_SPDT_RAYEX-L90, symbol Relay:RAYEX-L90
- added L1: L, Inductor_SMD:L_0805_2012Metric, symbol Device:L
- added Q1: BC337, Package_TO_SOT_THT:TO-92_Inline, symbol Transistor_BJT:BC337
- added Q2: 2N2219, Package_TO_SOT_THT:TO-92L_Inline, symbol Transistor_BJT:2N2219
- added Q3: 2N3905, Package_TO_SOT_THT:TO-92_Inline, symbol Transistor_BJT:2N3905
- added R1: 470k, Resistor_SMD:R_0201_0603Metric, symbol Device:R
- added R10, R12, R5: 10K, Resistor_SMD:R_0201_0603Metric, symbol Device:R
- added R11, R13, R3: 10k, Resistor_SMD:R_0201_0603Metric, symbol Device:R
- added R2: 5k, Resistor_SMD:R_0201_0603Metric, symbol Device:R
- added R4: 4.2K, Resistor_SMD:R_0201_0603Metric, symbol Device:R
- added R6, R7: 220, Resistor_SMD:R_0201_0603Metric, symbol Device:R
- added R8: 8K, Resistor_SMD:R_0201_0603Metric, symbol Device:R
- added R9: 2K, Resistor_SMD:R_0201_0603Metric, symbol Device:R
- added SW1: SW_Push, Button_Switch_SMD:SW_SPST_TS-1088-xR020, symbol Switch:SW_Push
- added U1: LM2596S-5V, Package_TO_SOT_SMD:TO-263-5_TabPin3, symbol Regulator_Switching:LM2596S-5
- added U2: LM358, Package_SO:SOIC-8-1EP_3.9x4.9mm_P1.27mm_EP2.29x3mm, symbol Amplifier_Operational:LM358
- added U2-TPS71533__SC70: U2 - 3,3V, Package_TO_SOT_SMD:SOT-353_SC-70-5, symbol Regulator_Linear:TPS71533__SC70
- added U3: ACS781xLRTR-050B, Sensor_Current:Allegro_PSOF-7_4.8x6.4mm_P1.60mm, symbol Sensor_Current:ACS781xLRTR-050B
- added U4: LM339, Package_TO_SOT_SMD:SOT-23-6, symbol Comparator:LM339
- added U5: 4013, Package_DIP:DIP-14_W7.62mm, symbol 4xxx:4013
- added U7: TEN20-4823WIN, Converter_DCDC:Converter_DCDC_TRACO_TEN20-xxxx_THT, symbol Converter_DCDC:TEN20-4823WIN
- added U8: AD633JRZ-R7, Package_SO:SOIC-8-1EP_3.9x4.9mm_P1.27mm_EP2.29x3mm, symbol AD633JRZ-R7:AD633JRZ-R7
- C1: value 1F -> 680uF; footprint Capacitor_SMD:C_0805_2012Metric -> Capacitor_SMD:C_0402_1005Metric
Connections:
- net at C1.1: now also J2.2 (Pin_2), U1.1 (VIN); no longer C1.2
- new net: J3.1 (Pin_1), K1.14
- new net: J3.2 (Pin_2), K1.11A, K1.11B
- new net: R2.2, R4.1, SW1.1, U4.4 (-)
- new net: R5.1, SW1.2, U5.4 (R)
- new net: C4.2, U2-TPS71533__SC70.5 (OUT), U3.1 (VCC)
- new net: Q1.2 (B), Q2.2 (B), Q3.2 (B), U5.2 (~{Q})
- new net: D2.1 (K), Q2.3 (C)
- new net: D1.1 (K), L1.1, U1.2 (OUT)
- new net: R1.2, U4.2, U5.6 (S)
- new net: R10.1, R11.1, U2.2 (-)
- new net: R8.1, R9.2, U8.7 (X1)
- new net: U7.3 (VOUT+), U8.6 (+VS)
- new net: U7.5 (VOUT-), U8.3 (-VS)
- new net: D3.1 (K), Q3.3 (C)
- new net: D4.1 (K), J4.1 (Pin_1), K1.A1
- new net: J1-ALLEGRO1.1 (Pin_1), U3.6 (IP-)
- new net: J1-ALLEGRO1.2 (Pin_2), U3.5 (IP+)
- new net: D2.2 (A), R6.2
- new net: D3.2 (A), R7.2
- new net: R12.2, R13.1, U2.3 (+)
- new net: R13.2, U2.1, U8.1 (Y1)
- new net: R3.1, U5.1 (Q)
- new net: D4.2 (A), K1.A2, Q1.1 (C)
- new net 24/48 V: J5.2 (Pin_2), R8.2, U7.1 (VIN+)
- new net 5V: C2.1, L1.2, R2.1, R6.1, R7.1, U1.4 (FB), U2-TPS71533__SC70.4 (IN)
- new net GND: C1.2, C2.2, C3.2, C4.1, D1.2 (A), J2.1 (Pin_1), J4.2 (Pin_2), J5.1 (Pin_1), K1.12, Q1.3 (E), Q2.1 (E), Q3.1 (E), R10.2, R11.2, R3.2, R4.2, R5.2, R9.1, U1.3 (GND), U1.5 (~{ON}/OFF), U2-TPS71533__SC70.2 (GND), U3.2 (GND), U3.4 (NC), U3.7 (NC), U5.3 (C), U5.5 (D), U7.2 (VIN-), U7.4 (CM), U8.2 (Y2), U8.4 (Z), U8.8 (X2)
- new net U2A: C3.1, U3.3 (VOUT)
- new net U3: R12.1
- new net U4A: U8.5 (W)
- new net U8: R1.1, U4.5 (+)
Other:
- note added: "9/17 V"
